File: hardware/source/carrier_board/carrier_board.kicad_sch (KiCad schematic)
At the start: 23 parts, among them J1 12V_CAR_IN, J2 JST_PH_LIPO, J3 LUCKFOX_J1_LEFT, J4 LUCKFOX_J2_RIGHT, J5 SC3336_MIPI_FPC, J7 USB_WIFI_PORT, SW1 MODE_SW, U1 LM2596_BUCK, U2 IP5306_BMS

Commit message: Fix schematic layout: migrate to A3, eliminate overlapping labels, clean functional zones
Connections:
- net +3V3: no longer C1.2, C2.2, C3.2, C6.2, C7.2, C8.2, C9.2, D1.2 (A), D2.2 (K), J1.2 (Pin_2), J3.3 (Pin_3), J3.7 (Pin_7), J4.2 (Pin_2), J4.8 (Pin_8), J5.1 (Pin_1), J5.10 (Pin_10), J5.4 (Pin_4), J5.7 (Pin_7), J7.4 (Pin_4), SW1.2, U1.2 (IN-), U1.4 (OUT-), U2.4 (GND)
- net GND: now reaches D2.1 (A), R3.2
- net GND: now also C1.2, C2.2, C3.2, C6.2, C7.2, C8.2, C9.2, D1.2 (A), D2.2 (K), J1.2 (Pin_2), J3.3 (Pin_3), J3.7 (Pin_7), J4.2 (Pin_2), J4.8 (Pin_8), J5.1 (Pin_1), J5.10 (Pin_10), J5.4 (Pin_4), J5.7 (Pin_7), J7.4 (Pin_4), SW1.2, U1.2 (IN-), U1.4 (OUT-), U2.4 (GND)
Other:
- note added: "- Connectivity: RTL8188EUS 2.4GHz 802.11b/g/n USB Wi-Fi"
- note added: "- Form Factor: 65.0 x 42.0 mm (Matching Luckfox Pico Mini B)"
- note added: "- PCB Spec: 2-Layer FR4, 1.6mm thickness, 1oz copper"
- note added: "- Power Input: 12V-24V Car Accessory Socket via LM2596 Buck"
- note added: "- Sensor: SmartSens SC3336 3MP CMOS (2304x1296 @ 30fps)"
- note added: "- SoC: Rockchip RV1103 (Cortex-A7 @ 1.2GHz + 0.5TOPS NPU)"
- note added: "- UPS Buffer: IP5306 + 3.7V 1000mAh LiPo (Safe shutdown)"
- note added: "- Video: Hardware H.264/H.265 encoder via RTSP streaming"
- note added: "15-Pin 0.5mm FPC (2-Lane MIPI + I2C)"
- note added: "DASHCAM PROTOTYPE ARCHITECTURE SUMMARY"
- note added: "Dual 8-Pin 2.54mm pitch female header sockets (J3 Left / J4 Right)"
- note added: "Host port for RTL8188EUS Wi-Fi dongle, Mode Tactile Switch & Status LED"
- note added: "Pre-regulates 12V automotive power to +5V_PRE (2A capacity)"
- note added: "SECTION 1: AUTOMOTIVE 12V-24V INPUT & LM2596 BUCK PRE-REGULATOR"
- note added: "SECTION 2: IP5306 BMS & 3.7V LIPO BATTERY BUFFER"
- note added: "SECTION 3: LUCKFOX PICO MINI B (RV1103) SBC EXPANSION SOCKETS"
- note added: "SECTION 4: USB 2.0 WI-FI DONGLE PORT & USER CONTROLS"
- note added: "SECTION 5: SC3336 CAMERA MIPI CSI-2"
- note added: "Seamless UPS power path: Charges 1000mAh LiPo & boosts to +5V_SYS"
- note removed: "1. AUTOMOTIVE 12V INPUT & LM2596 BUCK PRE-REGULATOR"
- note removed: "2. IP5306 BMS & 3.7V LIPO BATTERY BUFFER"
- note removed: "3. LUCKFOX PICO MINI B SBC SOCKETS"
- note removed: "4. USB WI-FI PORT & USER INTERFACE"
- note removed: "5. SMARTSENS SC3336 3MP CAMERA 15-PIN FPC"

Commit message: Fix carrier board schematic text alignment, net labels, and component routing
- Add left justification to section headers and architecture notes so text stays within dashed block boundaries
- Align net labels above horizontal wires with proper endpoint anchors and group connector GND pins onto vertical buses for J3, J4, and J5
- Adjust component reference/value justifications and offsets to prevent overlap with symbols and vertical wires
- Fix wire routing around J1, J2, C5, J7, C9, SW1, and D2 so wires connect cleanly to pin terminals
- Add missing power:+12V symbol definition and increase power symbol label clearances
- Regenerate carrier_board.kicad_sch, SVG, PDF, and high-resolution PNG preview
Connections:
- net GND: now also C4.2, C5.2, J2.2 (Pin_2), R1.2; no longer D2.1 (A), R3.2
- net VBAT: now also C5.1, J2.1 (Pin_1), U2.2 (BAT+)
- net +12V: now reaches C1.1, D1.1 (K), J1.1 (Pin_1), U1.1 (IN+)
- new net: D2.1 (A), R3.2
